File: Tri-color LED Breakout-v13.sch (EAGLE design)
At the start: 20 parts, among them Q1 2N3904, Q2 2N3904, Q3 2N3904

Commit message: Added OSHW logo to board. Added BOM.
Parts:
- added U$6: OSHW-LOGOS, SparkFun-Aesthetics:OSHW-LOGOS
Changed lines of the file:
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@@
 <layer number="121" name="_tsilk" color="7" fill="1" visible="yes" active="yes"/>
 <layer number="122" name="_bsilk" color="7" fill="1" visible="yes" active="yes"/>
+<layer number="125" name="_tNames" color="7" fill="1" visible="no" active="yes"/>
+<layer number="144" name="Drill_legend" color="7" fill="1" visible="no" active="yes"/>
 <layer number="151" name="HeatSink" color="7" fill="1" visible="yes" active="yes"/>
 <layer number="200" name="200bmp" color="1" fill="10" visible="yes" active="yes"/>
@@
 <layer number="207" name="207bmp" color="8" fill="10" visible="yes" active="yes"/>
 <layer number="208" name="208bmp" color="9" fill="10" visible="yes" active="yes"/>
+<layer number="209" name="209bmp" color="7" fill="1" visible="no" active="yes"/>
+<layer number="210" name="210bmp" color="7" fill="1" visible="no" active="yes"/>
+<layer number="211" name="211bmp" color="7" fill="1" visible="no" active="yes"/>
+<layer number="212" name="212bmp" color="7" fill="1" visible="no" active="yes"/>
+<layer number="213" name="213bmp" color="7" fill="1" visible="no" active="yes"/>
+<layer number="214" name="214bmp" color="7" fill="1" visible="no" active="yes"/>
+<layer number="215" name="215bmp" color="7" fill="1" visible="no" active="yes"/>
+<layer number="216" name="216bmp" color="7" fill="1" visible="no" active="yes"/>
+<layer number="217" name="217bmp" color="18" fill="1" visible="no" active="no"/>
+<layer number="218" name="218bmp" color="19" fill="1" visible="no" active="no"/>
+<layer number="219" name="219bmp" color="20" fill="1" visible="no" active="no"/>
+<layer number="220" name="220bmp" color="21" fill="1" visible="no" active="no"/>
+<layer number="221" name="221bmp" color="22" fill="1" visible="no" active="no"/>
+<layer number="222" name="222bmp" color="23" fill="1" visible="no" active="no"/>
+<layer number="223" name="223bmp" color="24" fill="1" visible="no" active="no"/>
+<layer number="224" name="224bmp" color="25" fill="1" visible="no" active="no"/>
 <layer number="250" name="Descript" color="3" fill="1" visible="no" active="no"/>
 <layer number="251" name="SMDround" color="12" fill="11" visible="no" active="no"/>
@@
 <part name="JP3" library="SparkFun" deviceset="STAND-OFF" device=""/>
 <part name="JP7" library="SparkFun" deviceset="LOGO-SFE" device="SK"/>
+<part name="U$6" library="SparkFun-Aesthetics" deviceset="OSHW-LOGO" device="S"/>
 </parts>
 <sheets>
@@
 <instance part="JP3" gate="G$1" x="241.3" y="30.48"/>
 <instance part="JP7" gate="G$1" x="231.14" y="17.78"/>
+<instance part="U$6" gate="G$1" x="132.08" y="10.16"/>
 </instances>
 <busses>

Commit message: Protos works. Added measurements to schematic.
Other:
- note added: "63.6mA"
- note added: "68.3mA"
- note added: "73.4mA"
- note added: "Measurements @ 5V:"
Changed lines of the file:
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@@
 <text x="22.86" y="127" size="1.778" layer="97">Part: 22QBK-ND</text>
 <text x="22.86" y="116.84" size="1.778" layer="97">Part: 22QBK-ND</text>
+<text x="50.8" y="78.74" size="1.778" layer="97">Measurements @ 5V:</text>
+<text x="86.36" y="78.74" size="1.778" layer="97">73.4mA</text>
+<text x="124.46" y="78.74" size="1.778" layer="97">63.6mA</text>
+<text x="162.56" y="78.74" size="1.778" layer="97">68.3mA</text>
 </plain>
 <instances>
